File: 2020/ele_cad/amano/em920/em920_remote/em920_remote.sch (KiCad schematic (older format))
At the start: 13 parts, among them SW1 SW_Push, U1 ATtiny85-20PU, U2 TY92SS, U3 LP2950-3.3_TO92

Commit message: em920の更新
Parts:
- removed D3: DIODE, Diode_THT:D_A-405_P7.62mm_Horizontal, symbol pspice:DIODE
- removed U3: LP2950-3.3_TO92, Package_TO_SOT_THT:TO-92_Inline_Wide, symbol Regulator_Linear:LP2950-3.3_TO92
- added IC1: NJM2391DL1-33-TE1, TO-252-3-L1, symbol em920:NJM2391DL1-33-TE1
- C1: value 0.33uF -> 0.1uF
- C2: value 2.2uF -> 10uF
Connections:
- wire segments 50 -> 44
Other:
- moved on the sheet: BT1, C1, C2
Changed lines of the file:
@@
 L power:GND #PWR010
 U 1 1 60FEC894
-P 1000 3700
-F 0 "#PWR010" H 1000 3450 50  0001 C CNN
-F 1 "GND" H 1005 3527 50  0000 C CNN
-F 2 "" H 1000 3700 50  0001 C CNN
-F 3 "" H 1000 3700 50  0001 C CNN
-	1    1000 3700
+P 900 3550
+F 0 "#PWR010" H 900 3300 50  0001 C CNN
+F 1 "GND" H 905 3377 50  0000 C CNN
+F 2 "" H 900 3550 50  0001 C CNN
+F 3 "" H 900 3550 50  0001 C CNN
+	1    900  3550
 	1    0    0    -1
 $EndComp
@@
 L Device:Battery_Cell BT1
 U 1 1 60FEA297
-P 1000 3400
-F 0 "BT1" H 1118 3496 50  0000 L CNN
-F 1 "Battery_Cell" H 1118 3405 50  0000 L CNN
-F 2 "Connector_PinHeader_2.54mm:PinHeader_1x03_P2.54mm_Vertical" V 1000 3460 50  0001 C CNN
-F 3 "~" V 1000 3460 50  0001 C CNN
-	1    1000 3400
+P 900 3250
+F 0 "BT1" H 1018 3346 50  0000 L CNN
+F 1 "Battery_Cell" H 1018 3255 50  0000 L CNN
+F 2 "Connector_PinHeader_2.54mm:PinHeader_1x03_P2.54mm_Vertical" V 900 3310 50  0001 C CNN
+F 3 "~" V 900 3310 50  0001 C CNN
+	1    900  3250
 	1    0    0    -1
 $EndComp
@@
 	1    0    0    -1
 $EndComp
-$Comp
-L Device:C C1
-U 1 1 60FF4567
-P 2350 3550
-F 0 "C1" H 2500 3600 50  0000 L CNN
-F 1 "0.33uF" H 2500 3550 50  0000 L CNN
-F 2 "Capacitor_THT:C_Disc_D3.0mm_W1.6mm_P2.50mm" H 2388 3400 50  0001 C CNN
-F 3 "~" H 2350 3550 50  0001 C CNN
-F 4 "Capacitor_THT:C_Disc_D3.0mm_W1.6mm_P2.50mm" H 2350 3550 50  0001 C CNN "Footprint"
-F 5 "C1" H 2350 3550 50  0001 C CNN "Value"
-	1    2350 3550
-	1    0    0    -1
-$EndComp
-Wire Wire Line
-	1000 3500 1000 3700
-Wire Wire Line
-	1000 3100 1000 3200
+Wire Wire Line
+	900  3350 900  3550
+Wire Wire Line
+	900  2950 900  3050
 $Comp
 L power:+BATT #PWR0101
 U 1 1 60FED62E
-P 1000 3100
-F 0 "#PWR0101" H 1000 2950 50  0001 C CNN
-F 1 "+BATT" H 1015 3273 50  0000 C CNN
-F 2 "" H 1000 3100 50  0001 C CNN
-F 3 "" H 1000 3100 50  0001 C CNN
-	1    1000 3100
+P 900 2950
+F 0 "#PWR0101" H 900 2800 50  0001 C CNN
+F 1 "+BATT" H 915 3123 50  0000 C CNN
+F 2 "" H 900 2950 50  0001 C CNN
+F 3 "" H 900 2950 50  0001 C CNN
+	1    900  2950
 	1    0    0    -1
 $EndComp
@@
 	6100 3550 6500 3550
 $Comp
-L power:+3V3 #PWR012
-U 1 1 6101B33D
-P 3900 3100
-F 0 "#PWR012" H 3900 2950 50  0001 C CNN
-F 1 "+3V3" H 3915 3273 50  0000 C CNN
-F 2 "" H 3900 3100 50  0001 C CNN
-F 3 "" H 3900 3100 50  0001 C CNN
-	1    3900 3100
-	1    0    0    -1
-$EndComp
-$Comp
 L em920:TY92SS U2
 U 1 1 61021B87
@@
 F 3 "" H 7300 3350 50  0001 C CNN
 	1    7300 3350
-	1    0    0    -1
-$EndComp
-$Comp
-L power:+BATT #PWR09
-U 1 1 6101B870
-P 2000 3100
-F 0 "#PWR09" H 2000 2950 50  0001 C CNN
-F 1 "+BATT" H 2015 3273 50  0000 C CNN
-F 2 "" H 2000 3100 50  0001 C CNN
-F 3 "" H 2000 3100 50  0001 C CNN
-	1    2000 3100
 	1    0    0    -1
 $EndComp
@@
 NoConn ~ 8200 3800
 Wire Wire Line
-	2000 3200 2350 3200
-$Comp
-L Regulator_Linear:LP2950-3.3_TO92 U3
-U 1 1 6120B41F
-P 3000 3200
-F 0 "U3" H 3000 3442 50  0000 C CNN
-F 1 "LP2950-3.3_TO92" H 3000 3351 50  0000 C CNN
-F 2 "Package_TO_SOT_THT:TO-92_Inline_Wide" H 3000 3425 50  0001 C CIN
-F 3 "http://www.ti.com/lit/ds/symlink/lp2950-n.pdf" H 3000 3150 50  0001 C CNN
-	1    3000 3200
-	1    0    0    -1
-$EndComp
-Wire Wire Line
-	2000 3100 2000 3200
-Wire Wire Line
-	3300 3200 3650 3200
-Wire Wire Line
-	3900 3200 3900 3100
-$Comp
-L power:GND #PWR0103
-U 1 1 61217D47
-P 3000 3850
-F 0 "#PWR0103" H 3000 3600 50  0001 C CNN
-F 1 "GND" H 3005 3677 50  0000 C CNN
-F 2 "" H 3000 3850 50  0001 C CNN
-F 3 "" H 3000 3850 50  0001 C CNN
-	1    3000 3850
-	1    0    0    -1
-$EndComp
-Wire Wire Line
-	3000 3500 3000 3800
-$Comp
-L Device:C C2
-U 1 1 6122145A
-P 3650 3550
-F 0 "C2" H 3800 3600 50  0000 L CNN
-F 1 "2.2uF" H 3800 3550 50  0000 L CNN
-F 2 "Capacitor_THT:C_Disc_D3.0mm_W1.6mm_P2.50mm" H 3688 3400 50  0001 C CNN
-F 3 "~" H 3650 3550 50  0001 C CNN
-F 4 "Capacitor_THT:C_Disc_D3.0mm_W1.6mm_P2.50mm" H 3650 3550 50  0001 C CNN "Footprint"
-F 5 "C1" H 3650 3550 50  0001 C CNN "Value"
-	1    3650 3550
-	1    0    0    -1
-$EndComp
-Wire Wire Line
-	2350 3200 2350 3400
-Wire Wire Line
-	2350 3800 3000 3800
-Wire Wire Line
-	2350 3700 2350 3800
-Connection ~ 2350 3200
-Connection ~ 3000 3800
-Wire Wire Line
-	3000 3800 3000 3850
-Wire Wire Line
-	3000 3800 3650 3800
-Wire Wire Line
-	3650 3800 3650 3700
-$Comp
-L pspice:DIODE D3
-U 1 1 6122E5B9
-P 3000 2700
-F 0 "D3" H 3000 2435 50  0000 C CNN
-F 1 "DIODE" H 3000 2526 50  0000 C CNN
-F 2 "Diode_THT:D_A-405_P7.62mm_Horizontal" H 3000 2700 50  0001 C CNN
-F 3 "~" H 3000 2700 50  0001 C CNN
-	1    3000 2700
-	-1   0    0    1
-$EndComp
-Wire Wire Line
-	3650 3200 3650 2700
-Wire Wire Line
-	3650 2700 3200 2700
-Wire Wire Line
-	2350 2700 2350 3200
-Wire Wire Line
-	2800 2700 2350 2700
-Connection ~ 3650 3200
-Wire Wire Line
-	3650 3200 3900 3200
-Wire Wire Line
-	2350 3200 2700 3200
-Wire Wire Line
-	3650 3200 3650 3400
-Wire Wire Line
 	7150 3350 7150 3500
 Wire Wire Line
@@
 Wire Wire Line
 	6600 3250 6600 4550
+Wire Wire Line
+	2250 2900 2250 3000
+$Comp
+L power:+BATT #PWR09
+U 1 1 6101B870
+P 2250 2900
+F 0 "#PWR09" H 2250 2750 50  0001 C CNN
+F 1 "+BATT" H 2265 3073 50  0000 C CNN
+F 2 "" H 2250 2900 50  0001 C CNN
+F 3 "" H 2250 2900 50  0001 C CNN
+	1    2250 2900
+	1    0    0    -1
+$EndComp
+$Comp
+L power:GND #PWR0103
+U 1 1 61217D47
+P 3550 3850
+F 0 "#PWR0103" H 3550 3600 50  0001 C CNN
+F 1 "GND" H 3555 3677 50  0000 C CNN
+F 2 "" H 3550 3850 50  0001 C CNN
+F 3 "" H 3550 3850 50  0001 C CNN
+	1    3550 3850
+	1    0    0    -1
+$EndComp
+$Comp
+L em920:NJM2391DL1-33-TE1 IC1
+U 1 1 615752FD
+P 2450 3000
+F 0 "IC1" H 3000 3265 50  0000 C CNN
+F 1 "NJM2391DL1-33-TE1" H 3000 3174 50  0000 C CNN
+F 2 "TO-252-3-L1" H 3400 3100 50  0001 L CNN
+F 3 "https://www.njr.com/semicon/PDF/NJM2391_E.pdf" H 3400 3000 50  0001 L CNN
+F 4 "LDO Voltage Regulators LDO" H 3400 2900 50  0001 L CNN "Description"
+F 5 "513-NJM2391DL133-TE1" H 3400 2700 50  0001 L CNN "Mouser Part Number"
+F 6 "https://www.mouser.co.uk/ProductDetail/NJR/NJM2391DL1-33-TE1?qs=l%2FzmVEvW4JpmmNoqbD2bKw%3D%3D" H 3400 2600 50  0001 L CNN "Mouser Price/Stock"
+F 7 "New Japan Radio" H 3400 2500 50  0001 L CNN "Manufacturer_Name"
+F 8 "NJM2391DL1-33-TE1" H 3400 2400 50  0001 L CNN "Manufacturer_Part_Number"
+	1    2450 3000
+	1    0    0    -1
+$EndComp
+$Comp
+L power:+3V3 #PWR012
+U 1 1 6101B33D
+P 1700 2900
+F 0 "#PWR012" H 1700 2750 50  0001 C CNN
+F 1 "+3V3" H 1715 3073 50  0000 C CNN
+F 2 "" H 1700 2900 50  0001 C CNN
+F 3 "" H 1700 2900 50  0001 C CNN
+	1    1700 2900
+	1    0    0    -1
+$EndComp
+Wire Wire Line
+	2250 3650 2250 3800
+Wire Wire Line
+	3550 3800 3550 3850
+Connection ~ 3550 3800
+Wire Wire Line
+	2250 3800 3550 3800
+Wire Wire Line
+	3550 3000 3550 3800
+$Comp
+L Device:C C2
+U 1 1 6122145A
+P 1700 3500
+F 0 "C2" H 1850 3550 50  0000 L CNN
+F 1 "10uF" H 1850 3500 50  0000 L CNN
+F 2 "Capacitor_THT:C_Disc_D3.0mm_W1.6mm_P2.50mm" H 1738 3350 50  0001 C CNN
+F 3 "~" H 1700 3500 50  0001 C CNN
+F 4 "Capacitor_THT:C_Disc_D3.0mm_W1.6mm_P2.50mm" H 1700 3500 50  0001 C CNN "Footprint"
+F 5 "C1" H 1700 3500 50  0001 C CNN "Value"
+	1    1700 3500
+	1    0    0    -1
+$EndComp
+$Comp
+L Device:C C1
+U 1 1 60FF4567
+P 2250 3500
+F 0 "C1" H 2400 3550 50  0000 L CNN
+F 1 "0.1uF" H 2400 3500 50  0000 L CNN
+F 2 "Capacitor_THT:C_Disc_D3.0mm_W1.6mm_P2.50mm" H 2288 3350 50  0001 C CNN
+F 3 "~" H 2250 3500 50  0001 C CNN
+F 4 "Capacitor_THT:C_Disc_D3.0mm_W1.6mm_P2.50mm" H 2250 3500 50  0001 C CNN "Footprint"
+F 5 "C1" H 2250 3500 50  0001 C CNN "Value"
+	1    2250 3500
+	1    0    0    -1
+$EndComp
+Wire Wire Line
+	2250 3350 2250 3000
+Wire Wire Line
+	2250 3000 2450 3000
+Connection ~ 2250 3000
+Wire Wire Line
+	1700 3800 2250 3800
+Wire Wire Line
+	1700 2900 1700 3100
+Wire Wire Line
+	1700 3650 1700 3800
+Connection ~ 2250 3800
+Wire Wire Line
+	2450 3100 1700 3100
+Connection ~ 1700 3100
+Wire Wire Line
+	1700 3100 1700 3350
 $EndSCHEMATC
